File: mainboard.kicad_pcb (KiCad board)
At the start: 4 copper layers, 45 x 35 mm, 48 parts, among them IC1 BMX160, J1 Conn_01x01, J2 10118194-0001LF, J28 Conn_01x01, J29 Conn_01x01, J3 Micro_SD_Card, J30 Conn_01x01, J4 xf2m-2415-1a, J5 XF2M-1015-1A, SW1 KMR231NG LFS, U1 RFM95W-915S2, U2 ATSAMD51G_TQFN48, U3 DRV8848, U4 TPS82740BSIPR, U5 DRV8848, U6 MAX708RESA-T, U8 RFM95W-915S2, X1 ANTENNA_U.FL, X2 ANTENNA_U.FL

Commit message: Add files via upload
imported .dxf board outline from mechanical
Other:
- board size 45 x 35 mm -> 94.4 x 36.2 mm
Changed lines of the file:
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@@
-(kicad_pcb (version 20171130) (host pcbnew "(5.1.4)-1")
+(kicad_pcb (version 20171130) (host pcbnew "(5.1.4-0-10_14)")
   (general
     (thickness 1.2)
-    (drawings 35)
+    (drawings 47)
     (tracks 699)
     (zones 0)
@@
     )
   )
+  (gr_line (start 27.3168 107.247398) (end 27.3168 74.4474) (layer Edge.Cuts) (width 0.2))
+  (gr_line (start 28.916801 72.847399) (end 28.9168 74.4474) (layer Edge.Cuts) (width 0.2))
+  (gr_line (start 27.3168 74.4474) (end 28.9168 74.4474) (layer Edge.Cuts) (width 0.2))
+  (gr_line (start 72.5168 74.4474) (end 72.5168 107.247398) (layer Edge.Cuts) (width 0.2))
+  (gr_line (start 28.916801 108.847399) (end 70.9168 108.847399) (layer Edge.Cuts) (width 0.2))
+  (gr_line (start 28.916801 107.247398) (end 28.916801 108.847399) (layer Edge.Cuts) (width 0.2))
+  (gr_line (start 70.9168 72.847399) (end 28.916801 72.847399) (layer Edge.Cuts) (width 0.2))
+  (gr_line (start 72.5168 107.247398) (end 70.9168 107.247398) (layer Edge.Cuts) (width 0.2))
+  (gr_line (start 70.9168 108.847399) (end 70.9168 107.247398) (layer Edge.Cuts) (width 0.2))
+  (gr_line (start 28.916801 107.247398) (end 27.3168 107.247398) (layer Edge.Cuts) (width 0.2))
+  (gr_line (start 70.9168 74.4474) (end 72.5168 74.4474) (layer Edge.Cuts) (width 0.2))
+  (gr_line (start 70.9168 74.4474) (end 70.9168 72.847399) (layer Edge.Cuts) (width 0.2))
   (gr_line (start 116.7003 106.0416) (end 116.7003 109.0416) (layer Edge.Cuts) (width 0.15))
   (gr_line (start 116.7003 74.0416) (end 116.7003 77.0416) (layer Edge.Cuts) (width 0.15))
