File: mainboard.sch (KiCad schematic (older format))
At the start: 68 parts, among them J1 Conn_01x06, J2 USB_B_Micro, J3 xf2m-2415-1a, J4 XF2M-1015-1A, J5 Conn_01x02, J6 U.FL-R-SMT-1, Q1 RADFET, SW1 KMR231NG LFS, U1 BMX160, U10 TPS82740BSIPR, U2 MAX708RESA-T, U3 ATSAMD51J20A-M, U4 DRV8830DRC, U5 MR25H40, U6 DRV8830DRC, U7 ADS124S06IRHBR, U8 DRV8830DRC, U9 RFM98PW-symbols

Commit message: changed LDO and added RBF header
Parts:
- removed U10: TPS82740BSIPR, custom-footprints:TPS82740ASIPR, symbol mainboard-rescue:TPS82740ASIP-TPS82740-
- added C18, C19: 10uF, Capacitor_SMD:C_0402_1005Metric, symbol mainboard-rescue:C_Small-Device
- added C20: 1uF, Capacitor_SMD:C_0402_1005Metric, symbol mainboard-rescue:C_Small-Device
- added J7: Conn_02x02_Top_Bottom, Connector_PinSocket_1.27mm:PinSocket_2x02_P1.27mm_Vertical_SMD, symbol Connector_Generic:Conn_02x02_Top_Bottom
- added R6: 10K, Resistor_SMD:R_0402_1005Metric, symbol mainboard-rescue:R_US-Device
- added U11: AP2112K-3.3, Package_TO_SOT_SMD:SOT-23-5, symbol Regulator_Linear:AP2112K-3.3
- U3: symbol MCU_Microchip_SAMD:ATSAMD51J20A-M -> mainboard-rescue:ATSAMD51J20A-M-MCU_Microchip_SAMD
Connections:
- net +3V3: now also J7.1 (Pin_1)
- net BATT_P: now also J7.3 (Pin_3)
- net GND: now also C18.2, C19.2, C20.2, J7.4 (Pin_4), U11.2 (GND)
- net at D2.1 (K): now also C18.1, R6.1, U11.1 (VIN)
- new net: C19.1, C20.1, J7.2 (Pin_2), U11.5 (VOUT)
- new net: R6.2, U11.3 (EN)
- no-connect marks 10 -> 9
Other:
- note added: "Remove\nBefore\nFlight"
- note removed: "3.3V OUTPUT\nVSEL1=1\nVSEL2=1\nVSEL3=1"
- moved on the sheet: D2
Changed lines of the file:
@@
 Text GLabel 2400 8200 0    59   Output ~ 0
 SCK
-$Comp
-L mainboard-rescue:TPS82740ASIP-TPS82740- U10
-U 1 1 5C405342
-P 15550 2350
-F 0 "U10" H 15550 3000 60  0000 C CNN
-F 1 "TPS82740BSIPR" H 15550 2900 60  0000 C CNN
-F 2 "custom-footprints:TPS82740ASIPR" H 15550 2290 60  0001 C CNN
-F 3 "" H 15550 2350 60  0000 C CNN
-	1    15550 2350
-	1    0    0    -1
-$EndComp
-Wire Wire Line
-	16100 1950 16250 1950
-Wire Wire Line
-	16250 1950 16250 1900
-$Comp
-L mainboard-rescue:VUSB-power- #PWR069
-U 1 1 5C4E0F8E
-P 14500 1750
-F 0 "#PWR069" H 14500 1600 50  0001 C CNN
-F 1 "VUSB" H 14515 1923 50  0000 C CNN
-F 2 "" H 14500 1750 50  0001 C CNN
-F 3 "" H 14500 1750 50  0001 C CNN
-	1    14500 1750
-	1    0    0    -1
-$EndComp
-Connection ~ 14850 2150
-Wire Wire Line
-	14950 1950 14850 1950
-Wire Wire Line
-	14950 2750 14850 2750
-Wire Wire Line
-	14950 2550 14850 2550
-Connection ~ 14850 2550
-Text Notes 15350 2400 0    50   ~ 0
-3.3V OUTPUT\nVSEL1=1\nVSEL2=1\nVSEL3=1
-Wire Wire Line
-	16100 2700 16250 2700
-Wire Wire Line
-	14500 1750 14500 1950
-Wire Wire Line
-	14500 1950 14550 1950
 Text Notes 2600 5950 0    197  ~ 0
 SAMD51\n
-Wire Wire Line
-	14850 2150 14850 2550
-$Comp
-L power:+3V3 #PWR072
-U 1 1 5D24BB79
-P 16250 1900
-F 0 "#PWR072" H 16250 1750 50  0001 C CNN
-F 1 "+3V3" H 16265 2073 50  0000 C CNN
-F 2 "" H 16250 1900 50  0001 C CNN
-F 3 "" H 16250 1900 50  0001 C CNN
-	1    16250 1900
-	1    0    0    -1
-$EndComp
 $Comp
 L power:+3V3 #PWR023
@@
 	1    0    0    -1
 $EndComp
-Wire Wire Line
-	16100 2950 16250 2950
 $Comp
 L power:GND #PWR06
@@
 $EndComp
 $Comp
-L power:GND #PWR073
-U 1 1 5DB1D593
-P 16250 2950
-F 0 "#PWR073" H 16250 2700 50  0001 C CNN
-F 1 "GND" H 16255 2777 50  0000 C CNN
-F 2 "" H 16250 2950 50  0001 C CNN
-F 3 "" H 16250 2950 50  0001 C CNN
-	1    16250 2950
-	1    0    0    -1
-$EndComp
-Wire Wire Line
-	14850 2750 14850 2950
-Wire Wire Line
-	14850 2950 14950 2950
-Connection ~ 14850 2750
-Connection ~ 14850 1950
-$Comp
 L mainboard-rescue:C_Small-Device C6
 U 1 1 5D1C3FDB
@@
 	1    0    0    -1
 $EndComp
-Wire Wire Line
-	14850 1950 14850 2150
-Connection ~ 16250 2950
-Wire Wire Line
-	16250 2700 16250 2950
-Wire Wire Line
-	14950 2150 14850 2150
-NoConn ~ 16100 2450
 Text Notes 13600 9650 0    157  ~ 31
 mainboard v01
-Wire Wire Line
-	14850 2550 14850 2750
 $Comp
 L mainboard-rescue:BMX160-symbols U1
@@
 L mainboard-rescue:D_Schottky-Device D2
 U 1 1 5D1876FB
-P 14700 1950
-F 0 "D2" H 14700 1734 50  0000 C CNN
-F 1 "RB550V" H 14700 1825 50  0000 C CNN
-F 2 "Diode_SMD:D_SOD-323" H 14700 1950 50  0001 C CNN
-F 3 "~" H 14700 1950 50  0001 C CNN
-	1    14700 1950
-	-1   0    0    1
-$EndComp
-$Comp
-L power:GND #PWR04
-U 1 1 5F73E007
-P 6450 8300
-F 0 "#PWR04" H 6450 8050 50  0001 C CNN
-F 1 "GND" H 6455 8127 50  0000 C CNN
-F 2 "" H 6450 8300 50  0001 C CNN
-F 3 "" H 6450 8300 50  0001 C CNN
-	1    6450 8300
-	1    0    0    -1
+P 14100 1950
+F 0 "D2" V 14146 1871 50  0000 R CNN
+F 1 "RB550V" V 14055 1871 50  0000 R CNN
+F 2 "Diode_SMD:D_SOD-323" H 14100 1950 50  0001 C CNN
+F 3 "~" H 14100 1950 50  0001 C CNN
+	1    14100 1950
+	0    -1   -1   0
 $EndComp
 Wire Wire Line
@@
 $EndComp
 $Comp
-L MCU_Microchip_SAMD:ATSAMD51J20A-M U3
+L mainboard-rescue:ATSAMD51J20A-M-MCU_Microchip_SAMD U3
 U 1 1 5F37375A
 P 3150 8300
@@
 Wire Wire Line
 	1200 9000 1200 8650
+$Comp
+L power:GND #PWR0103
+U 1 1 5F4DBD34
+P 14100 2300
+F 0 "#PWR0103" H 14100 2050 50  0001 C CNN
+F 1 "GND" H 14100 2150 50  0000 C CNN
+F 2 "" H 14100 2300 50  0001 C CNN
+F 3 "" H 14100 2300 50  0001 C CNN
+	1    14100 2300
+	1    0    0    -1
+$EndComp
+$Comp
+L mainboard-rescue:C_Small-Device C20
+U 1 1 5F4DCCEC
+P 15600 2200
+F 0 "C20" H 15692 2246 50  0000 L CNN
+F 1 "1uF" H 15692 2155 50  0000 L CNN
+F 2 "Capacitor_SMD:C_0402_1005Metric" H 15600 2200 50  0001 C CNN
+F 3 "~" H 15600 2200 50  0001 C CNN
+	1    15600 2200
+	1    0    0    -1
+$EndComp
+$Comp
+L power:GND #PWR0104
+U 1 1 5F4DD69D
+P 15500 2300
+F 0 "#PWR0104" H 15500 2050 50  0001 C CNN
+F 1 "GND" H 15500 2150 50  0000 C CNN
+F 2 "" H 15500 2300 50  0001 C CNN
+F 3 "" H 15500 2300 50  0001 C CNN
+	1    15500 2300
+	1    0    0    -1
+$EndComp
+$Comp
+L Regulator_Linear:AP2112K-3.3 U11
+U 1 1 5F4E27CF
+P 14900 2200
+F 0 "U11" H 14900 2542 50  0000 C CNN
+F 1 "AP2112K-3.3" H 14900 2451 50  0000 C CNN
+F 2 "Package_TO_SOT_SMD:SOT-23-5" H 14900 2525 50  0001 C CNN
+F 3 "https://www.diodes.com/assets/Datasheets/AP2112.pdf" H 14900 2300 50  0001 C CNN
+	1    14900 2200
+	1    0    0    -1
+$EndComp
+Wire Wire Line
+	14600 2100 14300 2100
+$Comp
+L mainboard-rescue:C_Small-Device C18
+U 1 1 5F51EAFF
+P 14100 2200
+F 0 "C18" H 14009 2246 50  0000 R CNN
+F 1 "10uF" H 14009 2155 50  0000 R CNN
+F 2 "Capacitor_SMD:C_0402_1005Metric" H 14100 2200 50  0001 C CNN
+F 3 "~" H 14100 2200 50  0001 C CNN
+	1    14100 2200
+	1    0    0    -1
+$EndComp
+$Comp
+L mainboard-rescue:R_US-Device R6
+U 1 1 5F53229D
+P 14450 2200
+F 0 "R6" V 14337 2200 50  0000 C CNN
+F 1 "10K" V 14246 2200 50  0000 C CNN
+F 2 "Resistor_SMD:R_0402_1005Metric" V 14490 2190 50  0001 C CNN
+F 3 "~" H 14450 2200 50  0001 C CNN
+	1    14450 2200
+	0    -1   -1   0
+$EndComp
+Wire Wire Line
+	14300 2200 14300 2100
+Connection ~ 14300 2100
+Wire Wire Line
+	14300 2100 14100 2100
+$Comp
+L mainboard-rescue:C_Small-Device C19
+U 1 1 5F56CEE6
+P 15400 2200
+F 0 "C19" H 15309 2246 50  0000 R CNN
+F 1 "10uF" H 15309 2155 50  0000 R CNN
+F 2 "Capacitor_SMD:C_0402_1005Metric" H 15400 2200 50  0001 C CNN
+F 3 "~" H 15400 2200 50  0001 C CNN
+	1    15400 2200
+	1    0    0    -1
+$EndComp
+Wire Wire Line
+	15600 2100 15400 2100
+Connection ~ 15400 2100
+Wire Wire Line
+	15400 2100 15200 2100
+Wire Wire Line
+	15400 2300 15500 2300
+Connection ~ 15500 2300
+Wire Wire Line
+	15500 2300 15600 2300
+$Comp
+L mainboard-rescue:VUSB-power- #PWR0105
+U 1 1 5F5A77C3
+P 14100 1750
+F 0 "#PWR0105" H 14100 1600 50  0001 C CNN
+F 1 "VUSB" H 14115 1923 50  0000 C CNN
+F 2 "" H 14100 1750 50  0001 C CNN
+F 3 "" H 14100 1750 50  0001 C CNN
+	1    14100 1750
+	1    0    0    -1
+$EndComp
+Wire Wire Line
+	14100 1750 14100 1800
+Connection ~ 14100 2100
+$Comp
+L power:GND #PWR0106
+U 1 1 5F627C90
+P 14900 2500
+F 0 "#PWR0106" H 14900 2250 50  0001 C CNN
+F 1 "GND" H 14900 2350 50  0000 C CNN
+F 2 "" H 14900 2500 50  0001 C CNN
+F 3 "" H 14900 2500 50  0001 C CNN
+	1    14900 2500
+	1    0    0    -1
+$EndComp
+$Comp
+L power:+3V3 #PWR0107
+U 1 1 5F62E560
+P 15600 1750
+F 0 "#PWR0107" H 15600 1600 50  0001 C CNN
+F 1 "+3V3" H 15615 1923 50  0000 C CNN
+F 2 "" H 15600 1750 50  0001 C CNN
+F 3 "" H 15600 1750 50  0001 C CNN
+	1    15600 1750
+	1    0    0    -1
+$EndComp
+Wire Wire Line
+	15600 1750 15600 1950
+Wire Wire Line
+	15600 2050 15600 2100
+Connection ~ 15600 2100
+Text Notes 15950 1850 0    59   ~ 0
+Remove\nBefore\nFlight
+$Comp
+L Connector_Generic:Conn_02x02_Top_Bottom J7
+U 1 1 5F71412D
+P 15800 1950
+F 0 "J7" H 15850 1625 50  0000 C CNN
+F 1 "Conn_02x02_Top_Bottom" H 16200 2400 50  0001 C CNN
+F 2 "Connector_PinSocket_1.27mm:PinSocket_2x02_P1.27mm_Vertical_SMD" H 15800 1950 50  0001 C CNN
+F 3 "~" H 15800 1950 50  0001 C CNN
+	1    15800 1950
+	1    0    0    -1
+$EndComp
+Text GLabel 16100 1950 2    50   Input ~ 0
+BATT_P
+$Comp
+L power:GND #PWR0108
+U 1 1 5F728BA8
+P 16100 2050
+F 0 "#PWR0108" H 16100 1800 50  0001 C CNN
+F 1 "GND" H 16100 1900 50  0000 C CNN
+F 2 "" H 16100 2050 50  0001 C CNN
+F 3 "" H 16100 2050 50  0001 C CNN
+	1    16100 2050
+	1    0    0    -1
+$EndComp
 $EndSCHEMATC

Commit message: BATT_P cleanup. starting dosimeter tweaks
Connections:
- net ~DRDY is gone; now on net ADC_DRDY: U7.13 (DRDY_N)
- net RF_IO0: now reaches U9.6 (GPIO_0)
- net RF_IO0: now also U3.14 (PA05)
- net ADC_DRDY: now reaches U3.16 (PA07)
- net RF_BUSY: no longer names the net of U9.4 (GPIO_4)
- net RF_BUSY: no longer U3.14 (PA05)
Other:
- note added: "TODO\n- verify SERCOM\n- check fit in CAD\n- place fiducals"
- note added: "done"
- moved on the sheet: R7, R8
Changed lines of the file:
@@
 L mainboard-rescue:R_US-Device R8
 U 1 1 5DB33981
-P 1950 8350
-F 0 "R8" H 2050 8150 50  0000 C CNN
-F 1 "10K" H 2050 8250 50  0000 C CNN
-F 2 "Resistor_SMD:R_0402_1005Metric" V 1990 8340 50  0001 C CNN
-F 3 "~" H 1950 8350 50  0001 C CNN
-	1    1950 8350
+P 1850 8350
+F 0 "R8" H 1950 8150 50  0000 C CNN
+F 1 "10K" H 1950 8250 50  0000 C CNN
+F 2 "Resistor_SMD:R_0402_1005Metric" V 1890 8340 50  0001 C CNN
+F 3 "~" H 1850 8350 50  0001 C CNN
+	1    1850 8350
 	-1   0    0    1
 $EndComp
@@
 L mainboard-rescue:R_US-Device R7
 U 1 1 5DB33987
-P 1800 8450
-F 0 "R7" H 1700 8400 50  0000 C CNN
-F 1 "10K" H 1700 8500 50  0000 C CNN
-F 2 "Resistor_SMD:R_0402_1005Metric" V 1840 8440 50  0001 C CNN
-F 3 "~" H 1800 8450 50  0001 C CNN
-	1    1800 8450
+P 1700 8450
+F 0 "R7" H 1600 8400 50  0000 C CNN
+F 1 "10K" H 1600 8500 50  0000 C CNN
+F 2 "Resistor_SMD:R_0402_1005Metric" V 1740 8440 50  0001 C CNN
+F 3 "~" H 1700 8450 50  0001 C CNN
+	1    1700 8450
 	-1   0    0    1
 $EndComp
@@
 L power:+3V3 #PWR010
 U 1 1 5DB3398D
-P 1800 8200
-F 0 "#PWR010" H 1800 8050 50  0001 C CNN
-F 1 "+3V3" H 1815 8373 50  0000 C CNN
-F 2 "" H 1800 8200 50  0001 C CNN
-F 3 "" H 1800 8200 50  0001 C CNN
-	1    1800 8200
+P 1700 8200
+F 0 "#PWR010" H 1700 8050 50  0001 C CNN
+F 1 "+3V3" H 1715 8373 50  0000 C CNN
+F 2 "" H 1700 8200 50  0001 C CNN
+F 3 "" H 1700 8200 50  0001 C CNN
+	1    1700 8200
 	1    0    0    -1
 $EndComp
@@
 Text GLabel 3850 8400 2    50   BiDi ~ 0
 RF_RST
-Text GLabel 2450 7400 0    50   BiDi ~ 0
-RF_BUSY
 $Comp
 L mainboard-rescue:C_Small-Device C11
@@
 	1    0    0    -1
 $EndComp
-Text GLabel 1700 8600 0    59   BiDi ~ 0
+Text GLabel 1600 8600 0    59   BiDi ~ 0
 SDA2
-Text GLabel 1700 8500 0    59   BiDi ~ 0
+Text GLabel 1600 8500 0    59   BiDi ~ 0
 SCL2
 $Comp
@@
 	9450 5850 9450 6050
 Connection ~ 9450 6050
-Text GLabel 12600 5650 2    59   Output ~ 0
-~DRDY
-Wire Wire Line
-	12600 5650 12500 5650
 $Comp
 L Connector:TestPoint TP1
@@
 Text GLabel 14400 4750 0    50   BiDi ~ 0
 RF_RST
-Text GLabel 15600 4950 2    50   Output ~ 0
-RF_BUSY
 $Comp
 L power:GND #PWR070
@@
 ~RESET
 Wire Wire Line
-	1700 8600 1800 8600
-Wire Wire Line
-	1700 8500 1950 8500
-Wire Wire Line
-	1800 8600 2450 8600
-Connection ~ 1800 8600
-Wire Wire Line
-	1950 8500 2450 8500
-Connection ~ 1950 8500
-Wire Wire Line
-	1800 8200 1950 8200
-Wire Wire Line
-	1800 8300 1800 8200
-Connection ~ 1800 8200
-Text Notes 1400 8450 0    50   ~ 0
+	1600 8600 1700 8600
+Wire Wire Line
+	1600 8500 1850 8500
+Wire Wire Line
+	1700 8600 2450 8600
+Connection ~ 1700 8600
+Wire Wire Line
+	1850 8500 2450 8500
+Connection ~ 1850 8500
+Wire Wire Line
+	1700 8200 1850 8200
+Wire Wire Line
+	1700 8300 1700 8200
+Connection ~ 1700 8200
+Text Notes 1300 8450 0    50   ~ 0
 SERCOM1
 Text Notes 4850 8150 0    50   ~ 0
@@
 Wire Wire Line
 	3850 8200 4650 8200
-Text Notes 1900 7650 0    50   ~ 0
+Text Notes 1950 8050 1    50   ~ 0
 SERCOM0/2
 Text Notes 4650 9250 0    50   ~ 0
@@
 	1    0    0    -1
 $EndComp
+Text Notes 6400 4400 0    100  ~ 0
+TODO\n- verify SERCOM\n- check fit in CAD\n- place fiducals
+Text Notes 7700 4050 0    100  ~ 20
+done
+Text GLabel 14400 5250 0    50   BiDi ~ 0
+RF_IO0
+Text GLabel 2450 7400 0    50   BiDi ~ 0
+RF_IO0
+Text GLabel 2450 7600 0    50   Output ~ 0
+ADC_DRDY
+Text GLabel 12600 5650 2    50   Output ~ 0
+ADC_DRDY
+Wire Wire Line
+	12600 5650 12500 5650
 $EndSCHEMATC
