File: ant-breakout/ant breakout/ant breakout.sch (KiCad schematic (older format))
At the start: 3 parts, among them J1 Conn_Coaxial, U1 Balun

Commit message: updated footprint
Parts:
- J1: footprint Documents:SMA-J-P-H-ST-EM1_N -> SMA-J-P-H-RA-TH1:SAMTEC_SMA-J-P-H-RA-TH1
Changed lines of the file:
@@
 EESchema Schematic File Version 4
+LIBS:ant breakout-cache
 EELAYER 30 0
 EELAYER END
@@
 F 0 "J1" H 4750 3675 50  0000 L CNN
 F 1 "Conn_Coaxial" H 4750 3584 50  0000 L CNN
-F 2 "Documents:SMA-J-P-H-ST-EM1_N" H 4650 3700 50  0001 C CNN
+F 2 "SMA-J-P-H-RA-TH1:SAMTEC_SMA-J-P-H-RA-TH1" H 4650 3700 50  0001 C CNN
 F 3 " ~" H 4650 3700 50  0001 C CNN
 	1    4650 3700
