File: Motherboard/mainboard.sch (KiCad schematic (older format))
At the start: 48 parts, among them IC1 BMX160, J1 Conn_01x01, J2 10118194-0001LF, J28 Conn_01x01, J29 Conn_01x01, J3 Micro_SD_Card, J30 Conn_01x01, J4 xf2m-2415-1a, J5 XF2M-1015-1A, SW1 KMR231NG LFS, U1 RFM95W-915S2, U2 ATSAMD51G_TQFN48, U3 DRV8848, U4 TPS82740BSIPR, U5 DRV8848, U6 MAX708RESA-T, U8 RFM95W-915S2, X1 ANTENNA_U.FL, X2 ANTENNA_U.FL

Commit message: placement rework with 2019-10-23 mechanical updates
Parts:
- removed H1, H2, H3, H4: MountingHole, MountingHole:MountingHole_2.2mm_M2, symbol Mechanical:MountingHole
- removed X1, X2: ANTENNA_U.FL, Connector_Coaxial:U.FL_Molex_MCRF_73412-0110_Vertical, symbol mainboard-rescue:ANTENNA_U.FL-
- added C15: 0.1uF, Capacitor_SMD:C_0402_1005Metric, symbol mainboard-rescue:C_Small-Device
- added J? (x2): U.FL-R-SMT-1, custom-footprints:U.FL-R-SMT-1, symbol symbols:U.FL-R-SMT-1
Connections:
- wire segments 169 -> 165
Changed lines of the file:
@@
 $EndComp
-$Comp
-L Mechanical:MountingHole H4
-U 1 1 5DAAE797
-P 9850 6650
-F 0 "H4" H 9950 6696 50  0000 L CNN
-F 1 "MountingHole" H 9950 6605 50  0000 L CNN
-F 2 "MountingHole:MountingHole_2.2mm_M2" H 9850 6650 50  0001 C CNN
-F 3 "~" H 9850 6650 50  0001 C CNN
-	1    9850 6650
-	1    0    0    -1
-$EndComp
-$Comp
-L Mechanical:MountingHole H3
-U 1 1 5DAAFFA0
-P 9850 6450
-F 0 "H3" H 9950 6496 50  0000 L CNN
-F 1 "MountingHole" H 9950 6405 50  0000 L CNN
-F 2 "MountingHole:MountingHole_2.2mm_M2" H 9850 6450 50  0001 C CNN
-F 3 "~" H 9850 6450 50  0001 C CNN
-	1    9850 6450
-	1    0    0    -1
-$EndComp
-$Comp
-L Mechanical:MountingHole H1
-U 1 1 5DAB18C3
-P 8800 6450
-F 0 "H1" H 8700 6404 50  0000 R CNN
-F 1 "MountingHole" H 8700 6495 50  0000 R CNN
-F 2 "MountingHole:MountingHole_2.2mm_M2" H 8800 6450 50  0001 C CNN
-F 3 "~" H 8800 6450 50  0001 C CNN
-	1    8800 6450
-	-1   0    0    1
-$EndComp
-$Comp
-L Mechanical:MountingHole H2
-U 1 1 5DAB1C8C
-P 8800 6650
-F 0 "H2" H 8700 6604 50  0000 R CNN
-F 1 "MountingHole" H 8700 6695 50  0000 R CNN
-F 2 "MountingHole:MountingHole_2.2mm_M2" H 8800 6650 50  0001 C CNN
-F 3 "~" H 8800 6650 50  0001 C CNN
-	1    8800 6650
-	-1   0    0    1
-$EndComp
-$Comp
-L mainboard-rescue:ANTENNA_U.FL- X2
-U 1 1 5DAC9815
-P 10100 3900
-F 0 "X2" H 10150 3437 42  0000 C CNN
-F 1 "ANTENNA_U.FL" H 10150 3516 42  0000 C CNN
-F 2 "Connector_Coaxial:U.FL_Molex_MCRF_73412-0110_Vertical" H 10100 3900 50  0001 C CNN
-F 3 "" H 10100 3900 50  0001 C CNN
-	1    10100 3900
-	-1   0    0    1
-$EndComp
-$Comp
-L mainboard-rescue:ANTENNA_U.FL- X1
-U 1 1 5DACA8A6
-P 9100 5250
-F 0 "X1" H 9150 4787 42  0000 C CNN
-F 1 "ANTENNA_U.FL" H 9150 4866 42  0000 C CNN
-F 2 "Connector_Coaxial:U.FL_Molex_MCRF_73412-0110_Vertical" H 9100 5250 50  0001 C CNN
-F 3 "" H 9100 5250 50  0001 C CNN
-	1    9100 5250
-	-1   0    0    1
-$EndComp
-$Comp
-L power:GND #PWR01
-U 1 1 5DACFA75
-P 10350 3750
-F 0 "#PWR01" H 10350 3500 50  0001 C CNN
-F 1 "GND" H 10355 3577 50  0000 C CNN
-F 2 "" H 10350 3750 50  0001 C CNN
-F 3 "" H 10350 3750 50  0001 C CNN
-	1    10350 3750
-	1    0    0    -1
-$EndComp
-Wire Wire Line
-	10350 3750 10200 3750
-Wire Wire Line
-	10200 3750 10200 3700
-Connection ~ 10200 3700
-Wire Wire Line
-	10200 3700 10200 3600
-Wire Wire Line
-	8900 5250 8900 5150
-Wire Wire Line
-	8900 5150 8850 5150
-Wire Wire Line
-	9200 5050 9200 4950
-Wire Wire Line
-	9200 4800 9300 4800
-Connection ~ 9200 4950
-Wire Wire Line
-	9200 4950 9200 4800
-Connection ~ 9300 4800
 $Comp
 L mainboard-rescue:MAX708RESA-T-symbols U6
@@
 Text GLabel 10050 1350 2    50   Input ~ 0
 3V3
+$Comp
+L mainboard-rescue:C_Small-Device C15
+U 1 1 5DB6EC0C
+P 600 6850
+F 0 "C15" H 500 6950 50  0000 L CNN
+F 1 "0.1uF" H 350 6800 50  0000 L CNN
+F 2 "Capacitor_SMD:C_0402_1005Metric" H 600 6850 50  0001 C CNN
+F 3 "~" H 600 6850 50  0001 C CNN
+	1    600  6850
+	1    0    0    -1
+$EndComp
+Wire Wire Line
+	600  6750 750  6750
+Connection ~ 750  6750
+Wire Wire Line
+	750  6950 600  6950
+Connection ~ 750  6950
+$Comp
+L symbols:U.FL-R-SMT-1 J?
+U 1 1 5DBA79E5
+P 9450 5150
+F 0 "J?" H 9850 5415 50  0000 C CNN
+F 1 "U.FL-R-SMT-1" H 9850 5324 50  0000 C CNN
+F 2 "custom-footprints:U.FL-R-SMT-1" H 10100 5250 50  0001 L CNN
+F 3 "https://www.hirose.co.jp/cataloge_hp/ed_UFL_20141014.pdf" H 10100 5150 50  0001 L CNN
+F 4 "" H 10100 5050 50  0001 L CNN "Description"
+F 5 "" H 10100 4950 50  0001 L CNN "Height"
+F 6 "Hirose" H 10100 4850 50  0001 L CNN "Manufacturer_Name"
+F 7 "U.FL-R-SMT-1" H 10100 4750 50  0001 L CNN "Manufacturer_Part_Number"
+F 8 "" H 10100 4650 50  0001 L CNN "Mouser Part Number"
+F 9 "" H 10100 4550 50  0001 L CNN "Mouser Price/Stock"
+F 10 "" H 10100 4450 50  0001 L CNN "RS Part Number"
+F 11 "" H 10100 4350 50  0001 L CNN "RS Price/Stock"
+	1    9450 5150
+	1    0    0    -1
+$EndComp
+Wire Wire Line
+	9050 5150 8850 5150
+$Comp
+L symbols:U.FL-R-SMT-1 J?
+U 1 1 5DBBD914
+P 10400 3900
+F 0 "J?" H 10800 4165 50  0000 C CNN
+F 1 "U.FL-R-SMT-1" H 10800 4074 50  0000 C CNN
+F 2 "custom-footprints:U.FL-R-SMT-1" H 11050 4000 50  0001 L CNN
+F 3 "https://www.hirose.co.jp/cataloge_hp/ed_UFL_20141014.pdf" H 11050 3900 50  0001 L CNN
+F 4 "" H 11050 3800 50  0001 L CNN "Description"
+F 5 "" H 11050 3700 50  0001 L CNN "Height"
+F 6 "Hirose" H 11050 3600 50  0001 L CNN "Manufacturer_Name"
+F 7 "U.FL-R-SMT-1" H 11050 3500 50  0001 L CNN "Manufacturer_Part_Number"
+F 8 "" H 11050 3400 50  0001 L CNN "Mouser Part Number"
+F 9 "" H 11050 3300 50  0001 L CNN "Mouser Price/Stock"
+F 10 "" H 11050 3200 50  0001 L CNN "RS Part Number"
+F 11 "" H 11050 3100 50  0001 L CNN "RS Price/Stock"
+	1    10400 3900
+	1    0    0    -1
+$EndComp
+Wire Wire Line
+	10000 3900 9900 3900
+$Comp
+L power:GND #PWR?
+U 1 1 5DBC73C0
+P 9550 5450
+F 0 "#PWR?" H 9550 5200 50  0001 C CNN
+F 1 "GND" H 9555 5277 50  0000 C CNN
+F 2 "" H 9550 5450 50  0001 C CNN
+F 3 "" H 9550 5450 50  0001 C CNN
+	1    9550 5450
+	1    0    0    -1
+$EndComp
+$Comp
+L power:GND #PWR?
+U 1 1 5DBC75A7
+P 10500 4200
+F 0 "#PWR?" H 10500 3950 50  0001 C CNN
+F 1 "GND" H 10505 4027 50  0000 C CNN
+F 2 "" H 10500 4200 50  0001 C CNN
+F 3 "" H 10500 4200 50  0001 C CNN
+	1    10500 4200
+	1    0    0    -1
+$EndComp
 $EndSCHEMATC

Commit message: updated edge cuts to match updated mechanical .dxf file (to allow flat flex connectors to travel around board edge)
Parts:
- J? (x2): symbol symbols:U.FL-R-SMT-1 -> mainboard-rescue:U.FL-R-SMT-1-symbols
Changed lines of the file:
@@
 Connection ~ 750  6950
 $Comp
-L symbols:U.FL-R-SMT-1 J?
+L mainboard-rescue:U.FL-R-SMT-1-symbols J?
 U 1 1 5DBA79E5
 P 9450 5150
@@
 	9050 5150 8850 5150
 $Comp
-L symbols:U.FL-R-SMT-1 J?
+L mainboard-rescue:U.FL-R-SMT-1-symbols J?
 U 1 1 5DBBD914
 P 10400 3900

Commit message: updated pycubed board edge cuts, updated top layer copper edges, shifted USB card and flat flex connector (still need to shift camera connector)
Parts:
- removed D1: GREEN, LED_SMD:LED_0603_1608Metric, symbol mainboard-rescue:LED0805_NOOUTLINE-
- removed J1, J28, J29, J30: Conn_01x01, custom-footprints:castellated_small_1side, symbol mainboard-rescue:Conn_01x01-Connector_Generic
- removed J4: xf2m-2415-1a, custom-footprints:XF2M-2415-1A, symbol mainboard-rescue:xf2m-2415-1a-symbols
- added C16: 0.1uF, Capacitor_SMD:C_0402_1005Metric, symbol mainboard-rescue:C_Small-Device
- added D3: WS2812B, LED_SMD:LED_WS2812B_PLCC4_5.0x5.0mm_P3.2mm, symbol LED:WS2812B
- added FID1, FID2, FID3, FID4: Fiducial, custom-footprints:Fiducial_1mm_Silkscreen, symbol Mechanical:Fiducial
- added J1: Conn_01x06, Connector_PinHeader_1.27mm:PinHeader_2x03_P1.27mm_Vertical_SMD, symbol Connector_Generic:Conn_01x06
- added J4: xf2m-2415-1a, custom-footprints:XF2M-2415-1A, symbol symbols:xf2m-2415-1a
- added J9: Conn_01x02, Connector_PinHeader_2.54mm:PinHeader_1x02_P2.54mm_Vertical, symbol Connector_Generic:Conn_01x02
- added R10, R13, R9: 100K, Resistor_SMD:R_0402_1005Metric, symbol mainboard-rescue:R_US-Device
- added R11, R12: 0, Resistor_SMD:R_0402_1005Metric, symbol mainboard-rescue:R_US-Device
- added R14: 10K, Resistor_SMD:R_0402_1005Metric, symbol mainboard-rescue:R_US-Device
- J6, J7: renamed from J?; symbol mainboard-rescue:U.FL-R-SMT-1-symbols -> symbols:U.FL-R-SMT-1
- R1: value 330 -> 0
- renumbered IC1 to U7
Connections:
- net 3V3 is gone; now on net +3V3: C11.2, C13.2, U3.11 (VREF), U3.14 (VINT), U5.11 (VREF), U5.14 (VINT)
- net BATT_N is gone; now on net GND: J5.4
- net DAC0 is gone; now on net RF2_IO1: U2.3 (PA02/EINT2/AIN0/VOUT0)
- net MXZ_EN is gone; now on net M_EN: U3.1 (nSLEEP), U5.1 (nSLEEP)
- net PA04 is gone; now on net RF1_CS: U2.9 (PA04/I4/VREFB/AIN4/SERCOM0.0)
- net PA21 is gone; now on net M_FAULT: U2.30 (PA21/I5/SERCOM3+5.3/I2SDO)
- net PA22 is gone; now on net BURN1: U2.31 (PA22/I2C/I6/SERCOM3.0+5.1/I2SDI)
- net RF_CS is gone; now on net CS_CAM: U2.19 (PB10/I10/SERCOM4.2/I2SDI)
- net RX is gone; now on net RF1_RST: U2.8 (PB09/I9/AIN3/SERCOM4.1)
- net TX is gone; now on net RF2_RST: U2.7 (PB08/I8/AIN2/SERCOM4.0)
- net +3V3: now also U7.12 (CSB), C16.1, D3.1 (VDD), J1.1 (Pin_1), J4.12, J4.13, R13.2
- net BATT_P: now also J4.24, J9.2 (Pin_2), R9.2
- net BURN1: now also J4.7
- net BURN2: now also U2.29 (PA20/I4/SERCOM3+5.2/I2SFS0), J4.8
- net CS_CAM: now also J5.9; no longer J5.6, U2.24 (PA15/I15/SERCOM2+4.3)
- net CS_SD: now also U2.47 (PB02/I2/AIN14/SERCOM5.0)
- net EN_CAM: now also J5.8, U2.16 (PA11/I11/AIN11/SERCOM0+2.3/I2SDO); no longer J5.5, U2.29 (PA20/I4/SERCOM3+5.2/I2SFS0)
- net GND: now also C16.2, D3.3 (VSS), J1.3 (Pin_3), J4.14, J4.23, J9.1 (Pin_1), R10.1
- net MINX_1: now also U2.23 (PA14/I14/SERCOM2+4.2); no longer U5.16 (AIN1), U5.2 (AOUT1)
- net MINX_2: now also U2.22 (PA13/I13/I2C/SERCOM2.1+4.0); no longer U5.15 (AIN2), U5.4 (AOUT2)
- net MINZ_1: now also U2.20 (PB11/I11/SERCOM4.3/I2SFS1); no longer U5.9 (BIN1)
- net MINZ_2: now also U2.21 (PA12/I12/I2C/SERCOM2.0+4.1); no longer U5.10 (BIN2)
- net MISO: no longer U7.1 (SDO)
- net MOSI: now also J5.5; no longer J5.8, U7.14 (SDX)
- net RF2_BUSY: now also U2.39 (PA27/I11)
- net SCK: now also J5.6; no longer J5.9, U7.13 (SCX)
- net SCL1: now also U7.13 (SCX), J4.10
- net SCL2: now also J4.1
- net SDA1: now also U7.14 (SDX), J4.9
- net SDA2: now also J4.2
- net SWCLK: now also J1.4 (Pin_4)
- net SWDIO: now also J1.2 (Pin_2)
- net WDT_WDI: now also U2.38 (PB23/I7/SERCOM1+5.3); no longer U2.37 (PB22/I6/SERCOM1+5.2)
- net ~RESET: now also J1.5 (Pin_5)
- net at R1.1: now also J4.3
- net RF1_BUSY: now reaches U2.11 (PA06/I6/VREFC/AIN6/SERCOM0.2)
- net RF1_BUSY: now also U8.12 (DIO4)
- net M_EN: now reaches U2.28 (PA19/I3/SERCOM1+3.3)
- net RF2_IO1: now reaches U1.15 (DIO1)
- net CS_IMU renamed BATT_STATUS
- net BATT_STATUS: now also J4.11; no longer U7.12 (CSB)
- net CS_RF1 renamed RF1_CS
- net CS_RF2 renamed RF2_CS
- net RF2_CS: now also U2.48 (PB03/I3/AIN15/SERCOM5.1)
- net DAC1 renamed BATTERY
- net BATTERY: now also R10.2, R9.1
- net DXZ_FAULT renamed M_FAULT
- net M_FAULT: now also R13.1, R14.1; no longer U5.8 (nFAULT)
- net LED1: no longer names the net of R1.2
- net LED1: now also J4.5; no longer U2.48 (PB03/I3/AIN15/SERCOM5.1)
- net MOX_1 renamed COIL4_N
- net COIL4_N: now also J4.16
- net MOX_2 renamed COIL3_P
- net COIL3_P: now also J4.18
- net MOZ_1: no longer names the net of U5.7 (BOUT1)
- net MOZ_1: no longer U3.7 (BOUT1)
- net MOZ_2: no longer names the net of U5.5 (BOUT2)
- net MOZ_2: no longer U3.5 (BOUT2)
- net PA07 renamed RF1_IO1
- net RF1_IO1: now also U8.15 (DIO1)
- net PA23 renamed MINY_2
- net MINY_2: now also U5.15 (AIN2)
- removed net RF_BUSY: U2.22 (PA13/I13/I2C/SERCOM2.1+4.0), U8.12 (DIO4)
- net RF_DIO0: no longer names the net of U8.14 (DIO0)
- net RF_DIO0: no longer U2.47 (PB02/I2/AIN14/SERCOM5.0)
- removed net RF_DIO1: U2.39 (PA27/I11), U8.15 (DIO1)
- net RF_DIO2: no longer names the net of U8.16 (DIO2)
- net RF_DIO2: no longer U2.38 (PB23/I7/SERCOM1+5.3)
- net RF_DIO3: no longer names the net of U8.11 (DIO3)
- net RF_DIO3: no longer U2.23 (PA14/I14/SERCOM2+4.2)
- net RF_RST renamed RF1_RST
- net RF1_RST: no longer U2.21 (PA12/I12/I2C/SERCOM2.0+4.1)
- new net: D3.4 (DIN), U2.37 (PB22/I6/SERCOM1+5.2)
- new net: J4.19, R12.1
- new net: J4.21, R12.2
- new net: J4.15, R11.1
- new net: J4.17, R11.2
- new net COIL1_P: J4.22, U3.7 (BOUT1)
- new net COIL2_N: J4.20, U3.5 (BOUT2)
- new net COIL5_P: J4.6, U5.4 (AOUT2)
- new net COIL6_N: J4.4, U5.2 (AOUT1)
- new net MINY_1: U2.24 (PA15/I15/SERCOM2+4.3), U5.16 (AIN1)
- new net M_FAULT2: R14.2, U5.8 (nFAULT)
- no-connect marks 10 -> 11
Other:
- note added: "COIL1_N"
- note added: "COIL2_P"
- note added: "COIL3_N"
- note added: "COIL4_P"
- note added: "COIL5_N"
- note added: "COIL6_P"
- note added: "X"
- note added: "Y"
- note added: "Z"
- moved on the sheet: J5
